Commit message: added collisions

File: description/lidar.xacro (robot description, xacro)
@@ -13,4 +13,9 @@
             <material name="red"/>
         </visual>
+        <collision>
+            <geometry>
+                <cylinder radius="0.2" length="0.2"/>
+            </geometry>
+        </collision>
     </link>
     <gazebo reference="laser_frame">

File: description/robot_core.xacro (robot description, xacro)
@@ -27,5 +27,5 @@
         <parent link="base_link"/>
         <child link="chassis"/>
-        <origin xyz="-0.3 0 0"/>
+        <origin xyz="-0.3 0 0" rpy="0.0 0.0 0.0"/>
     </joint>
     <link name="chassis">
@@ -37,4 +37,10 @@
             <material name="white"/>
         </visual>
+        <collision>
+            <origin xyz="0.75 0 0.375"/>
+            <geometry>
+                <box size="${base_length} ${base_width} ${base_height}"/>
+            </geometry>
+        </collision>
     </link>
     <!-- left wheel -->
@@ -53,4 +59,9 @@
             <material name="blue"/>
         </visual>
+        <collision>
+            <geometry>
+                <cylinder radius="0.3" length="0.20"/>
+            </geometry>
+        </collision>
     </link>
     <gazebo reference="left_wheel">
@@ -71,4 +82,9 @@
             <material name="blue"/>
         </visual>
+        <collision>
+             <geometry>
+                <cylinder radius="0.3" length="0.20"/>
+            </geometry>
+        </collision>
     </link>
     <gazebo reference="right_wheel">
@@ -87,4 +103,9 @@
             <material name="black"/>
         </visual>
+        <collision>
+            <geometry>
+                <sphere radius="0.3"/>
+            </geometry>
+        </collision>
     </link>
     <gazebo reference="caster_wheel">
