Commit message: added gazebo control plugin

File: description/robot.urdf.xacro (robot description, xacro)
@@ -1,5 +1,7 @@
 <?xml version="1.0"?>
 <robot xmlns:xacro="http://www.ros.org/wiki/xacro"  name="robot">
+    <xacro:include filename="inertial_macros.xacro"/>
     <xacro:include filename="robot_core.xacro"/>
     <xacro:include filename="lidar.xacro"/>
+    <xacro:include filename="gazebo_control.xacro"/>
 </robot>

File: description/robot_core.xacro (robot description, xacro)
@@ -43,4 +43,7 @@
             </geometry>
         </collision>
+        <xacro:inertial_box mass="0.5" x="1.5" y="1.5" z="0.75">
+            <origin xyz="0.75 0 0.375" rpy="0 0 0"/>
+        </xacro:inertial_box>
     </link>
     <!-- left wheel -->
@@ -64,4 +67,7 @@
             </geometry>
         </collision>
+        <xacro:inertial_cylinder mass="0.1" length="0.2" radius="0.3">
+            <origin xyz="0 0 0" rpy="0 0 0"/>
+        </xacro:inertial_cylinder>
     </link>
     <gazebo reference="left_wheel">
@@ -87,4 +93,7 @@
             </geometry>
         </collision>
+        <xacro:inertial_cylinder mass="0.1" length="0.2" radius="0.3">
+            <origin xyz="0 0 0" rpy="0 0 0"/>
+        </xacro:inertial_cylinder>
     </link>
     <gazebo reference="right_wheel">
@@ -108,4 +117,7 @@
             </geometry>
         </collision>
+        <xacro:inertial_sphere mass="0.1" radius="0.3">
+            <origin xyz="0 0 0" rpy="0 0 0"/>
+        </xacro:inertial_sphere>
     </link>
     <gazebo reference="caster_wheel">
