Commit message: adding base_footprint for navigation&slam_toolbox

File: description/robot_core.xacro (robot description, xacro)
@@ -22,4 +22,13 @@
     <!-- base_link -->
      <link name="base_link">
+    </link>
+    <!-- Base footprint joint -->
+    <joint name="base_footprint_joint" type="fixed">
+        <parent link="base_link"/>
+        <child link="base_footprint"/>
+        <origin xyz="0.0 0.0 0.0" rpy="0.0 0.0 0.0"/>
+    </joint>
+    <!-- Base footprint link -->
+    <link name="base_footprint">
     </link>
     <!-- CHASSIS LINK -->
